Commit message: fix: removed --inorder from .urdf description; fix: added dummy link

File: kuka_kr16_support/urdf/kr16_2_macro.xacro (robot description, xacro)
@@ -4,4 +4,5 @@
     <!-- LINKS -->
     <!-- base link -->
+    <link name="dummy"/>
     <link name="${prefix}base_link">
       <inertial>
@@ -23,4 +24,8 @@
       </collision>
     </link>
+    <joint name="dummy_joint" type="fixed">
+     <parent link="dummy"/>
+     <child link="base_link"/>
+   </joint>
     <!-- link 1 (A1) -->
     <link name="${prefix}link_1">
