Commit message: refactor: implement robot and tool classes, and movement functions; fix: load model with tool correctly at roslaunch

File: kuka_kr16_support/urdf/kr16_2_with_tool_macro.xacro (robot description, xacro)
@@ -4,6 +4,6 @@
   <xacro:property name="tool_joint_offset" value="0.00 0.00 0.00" />
   <xacro:property name="tool_link_offset" value="0.00 0.00 0.354" />
-  <xacro:property name="marker_pen_offset" value="0.036 0.00 0.354" />
-  <xacro:property name="ballpoint_pen_offset" value="-0.036 0.00 0.354" />
+  <xacro:property name="marker_pen_offset" value="0.00 0.036 0.354" />
+  <xacro:property name="ballpoint_pen_offset" value="0.00 -0.036 0.354" />
   <xacro:macro name="kr16_2_with_tool" params="prefix">
     <!-- LINKS -->
@@ -159,5 +159,5 @@
       </inertial>
       <visual>
-        <origin xyz="0 0 0" rpy="0 0 0"/>
+        <origin xyz="0 0 0" rpy="0 0 ${radians(-90)}"/>
         <geometry>
 	      <mesh filename="package://kuka_kr16_support/meshes/kr16_2/visual/double_tool.dae"/>
@@ -165,5 +165,5 @@
       </visual>
       <collision>
-        <origin xyz="0 0 0" rpy="0 0 0"/>
+        <origin xyz="0 0 0" rpy="0 0 ${radians(-90)}"/>
           <geometry>
 	        <mesh filename="package://kuka_kr16_support/meshes/kr16_2/collision/double_tool.stl"/>
